File: test_power_step.kicad_sch (KiCad schematic)
At the start: 45 parts, among them J1 796636-6, J2 796636-2, J3 796636-4, J4 796634-6, J5 796634-2, J6 796634-4, Q1 ISZ015N04NM7V, Q2 ISZ015N04NM7V, SW1 SW_SPST, SW2 SW_SPST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

Commit message: update
Other:
- note added: "Step Resistors 3.3V, 0.6A, 5.6ohm, LTR100JZPF5R60 6.0V, 0.3A, 20ohm, LTR100JZPF20R0 16V, 0.05A, 330ohm, LTR100JZPF3300"
- note removed: "Step Resistors 3.3V, 0.6A, 5.6ohm, LTR100JZPF5R60 6.0V, 0.3A, 20ohm, LTR100JZPF20R0 16V, 0.05A, 320ohm, LTR100JZPF3300"
Changed lines of the file:
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@@
 		)
 	)
-	(text "Step Resistors\n3.3V, 0.6A, 5.6ohm, LTR100JZPF5R60\n6.0V, 0.3A, 20ohm, LTR100JZPF20R0\n16V, 0.05A, 320ohm, LTR100JZPF3300"
+	(text "Step Resistors\n3.3V, 0.6A, 5.6ohm, LTR100JZPF5R60\n6.0V, 0.3A, 20ohm, LTR100JZPF20R0\n16V, 0.05A, 330ohm, LTR100JZPF3300"
 		(exclude_from_sim no)
 		(at 40.894 123.19 0)
